Commit message: floating panda gripper

File: mani_skill/assets/robots/panda/panda_v2_gripper.urdf (robot description, URDF)
Before this commit: robot panda, 4 links, 3 joints
Links:
- added link root, mass 0
- added link root_arm_1_link_1, mass 0
- added link root_arm_1_link_2, mass 0
- added link root_arm_1_link_3, mass 0
- added link root_arm_1_link_4, mass 0
- added link root_arm_1_link_5, mass 0
Joints:
- added joint root_x_axis_joint: type prismatic, parent root, child root_arm_1_link_1, axis 1 0 0, limit lower=-20 upper=20 effort=100 velocity=0.50
- added joint root_x_rot_joint: type revolute, parent root_arm_1_link_3, child root_arm_1_link_4, axis 1 0 0, limit lower=-20 upper=20 effort=100 velocity=0.50
- added joint root_y_axis_joint: type prismatic, parent root_arm_1_link_1, child root_arm_1_link_2, axis 0 1 0, limit lower=-20 upper=20 effort=100 velocity=0.50
- added joint root_y_rot_joint: type revolute, parent root_arm_1_link_4, child root_arm_1_link_5, axis 0 1 0, limit lower=-20 upper=20 effort=100 velocity=0.50
- added joint root_z_axis_joint: type prismatic, parent root_arm_1_link_2, child root_arm_1_link_3, axis 0 0 1, limit lower=-20 upper=20 effort=100 velocity=0.50
- added joint root_z_rot_joint: type revolute, parent root_arm_1_link_5, child panda_hand, axis 0 0 1, limit lower=-20 upper=20 effort=100 velocity=0.50
